File: schematic/KiCad/wiring.kicad_sch (KiCad schematic)
At the start: 31 parts, among them SW1 Manual/Auto, SW2 Pulse, U1 74LS08, U10 74LS173, U11 74LS173, U12 74LS86, U13 74LS86, U14 74LS283, U15 74LS283, U16 74LS245, U2 74LS32, U3 NE555P, U4 NE555P, U5 NE555P, U6 74LS173, U7 74LS04, U8 74LS173, U9 74LS245

Commit message: Add files via upload
Parts:
- added R10, R2, R8, R9: 10K, symbol Device:R_Small
- added SW3: SW_DIP_x04, symbol Switch:SW_DIP_x04
- added U17: 74LS161, symbol 8-bit ICs:74LS161
- added U18, U19: 74LS245, symbol 8-bit ICs:74LS245
- added U20: 74LS173, symbol 8-bit ICs:74LS173
- added U22: 74LS157, symbol 8-bit ICs:74LS157
- added U23, U24: 74LS189, symbol 8-bit ICs:74LS189
- added U25, U26: 74LS04, symbol 8-bit ICs:74LS04
- added U27: 74LS00, symbol 8-bit ICs:74LS00
Connections:
- net +5V: now also SW3.1, SW3.2, SW3.3, SW3.4, U17.16 (VCC), U18.1 (DIR), U18.20 (VCC), U19.1 (DIR), U19.20 (VCC), U20.16 (VCC), U22.16 (VCC), U23.16 (VCC), U24.16 (VCC), U25.14 (VCC), U26.14 (VCC), U27.14 (VCC)
- net BUS1: now also U17.3 (A), U18.18 (B1), U19.18 (B1), U20.14 (1D), U23.4 (D1)
- net BUS2: now also U17.4 (B), U18.17 (B2), U19.17 (B2), U20.13 (2D), U23.6 (D2)
- net BUS3: now also U17.5 (C), U18.16 (B3), U19.16 (B3), U20.12 (3D), U23.10 (D3)
- net BUS4: now also U17.6 (D), U18.15 (B4), U19.15 (B4), U20.11 (4D), U23.12 (D4)
- net BUS5: now also U19.14 (B5), U24.4 (D1)
- net BUS6: now also U19.13 (B6), U24.6 (D2)
- net BUS7: now also U19.12 (B7), U24.10 (D3)
- net BUS8: now also U19.11 (B8), U24.12 (D4)
- net CLK: now also U17.2 (CLK), U20.7 (CLK), U27.1 (1A)
- net GND: now also R10.2, R2.2, R8.2, R9.2, U17.8 (GND), U18.10 (GND), U18.6 (A5), U18.7 (A6), U18.8 (A7), U18.9 (A8), U19.10 (GND), U20.8 (GND), U22.15 (ENABLE), U22.8 (GND), U23.2 (~{CS}), U23.8 (GND), U24.2 (~{CS}), U24.8 (GND), U25.7 (GND), U26.7 (GND), U27.7 (GND)
- new net: U17.14 (QA), U18.2 (A1)
- new net: U17.13 (QB), U18.3 (A2)
- new net: U17.12 (QC), U18.4 (A3)
- new net: U17.11 (QD), U18.5 (A4)
- new net: U20.10 (~{G2}), U20.9 (~{G1})
- new net CE: U17.10 (ENT), U17.7 (ENP)
- new net C_RST: U17.1 (~{CLR})
- new net JUMP: U17.9 (~{LOAD})
- new net MAR_RST: U20.15 (CLR)
- new net MUX1: U22.4 (Y1), U23.1 (A0), U24.1 (A0)
- new net MUX2: U22.7 (Y2), U23.15 (A1), U24.15 (A1)
- new net MUX3: U22.9 (Y3), U23.14 (A2), U24.14 (A2)
- new net MUX4: U22.12 (Y4), U23.13 (A3), U24.13 (A3)
- new net PROG1: R2.1, SW3.8, U22.3 (B1)
- new net PROG2: R8.1, SW3.7, U22.6 (B2)
- new net PROG3: R9.1, SW3.6, U22.10 (B3)
- new net PROG4: R10.1, SW3.5, U22.13 (B4)
- new net PROG/RUN: U22.1 (SELECT)
- new net RI: U27.2 (1B)
- new net RO: U19.19 (~{OE})
- new net RQ1: U20.3 (1Q), U22.2 (A1)
- new net RQ2: U20.4 (2Q), U22.5 (A2)
- new net RQ3: U20.5 (3Q), U22.11 (A3)
- new net RQ4: U20.6 (4Q), U22.14 (A4)
- new net SQ1: U19.2 (A1), U25.2 (1Y)
- new net SQ2: U19.3 (A2), U25.4 (2Y)
- new net SQ3: U19.4 (A3), U25.6 (3Y)
- new net SQ4: U19.5 (A4), U25.8 (4Y)
- new net SQ5: U19.6 (A5), U26.2 (1Y)
- new net SQ6: U19.7 (A6), U26.4 (2Y)
- new net SQ7: U19.8 (A7), U26.6 (3Y)
- new net SQ8: U19.9 (A8), U26.8 (4Y)
- new net WE: U23.3 (~{WE}), U24.3 (~{WE}), U27.3 (1Y)
- new net ~{C0}: U18.19 (~{OE})
- new net ~{MAR_I}: U20.1 (M), U20.2 (N)
- new net ~{SQ1}: U23.5 (~{Q1}), U25.1 (1A)
- new net ~{SQ2}: U23.7 (~{Q2}), U25.3 (2A)
- new net ~{SQ3}: U23.9 (~{Q3}), U25.5 (3A)
- new net ~{SQ4}: U23.11 (~{Q4}), U25.9 (4A)
- new net ~{SQ5}: U24.5 (~{Q1}), U26.1 (1A)
- new net ~{SQ6}: U24.7 (~{Q2}), U26.3 (2A)
- new net ~{SQ7}: U24.9 (~{Q3}), U26.5 (3A)
- new net ~{SQ8}: U24.11 (~{Q4}), U26.9 (4A)
- no-connect marks 21 -> 42
Other:
- note added: "16x8 SRAM Storage"
- note added: "Address MUX & Manual Control"
- note added: "Counter & Bus Output"
- note added: "MAR"
- note added: "Output Inverters"
- note added: "RAM & program counter"
- note added: "RAM Bus Transceiver"
- note added: "Write Pulse Logic"

Commit message: Add files via upload
Parts:
- added C10, C11, C12, C13, C14, C15, C16, C17, C18, C19, C20, C21, C22, C23, C24, C25, C26, C27, C28, C29, C3, C30, C31, C32, C33, C34, C35, C36, C37, C8, C9: 100nF, symbol Device:C_Small
- added C7: 10nF, symbol Device:C_Small
- added R11, R12, R13, R14, R15, R16, R17, R18: 330R, symbol Device:R_Small
- added R19: 1K, symbol Device:R_Small
- added R20: 10K, symbol Device:R_Small
- added U21: 74LS273, symbol 8-bit ICs:74LS273
- added U28: 28C16, symbol 8-bit ICs:28C16
- added U29: NE555P, Package_DIP:DIP-8_W7.62mm, symbol Timer:NE555P
- added U30: 74LS76, symbol 8-bit ICs:74LS76
- added U31: 74LS139, symbol 8-bit ICs:74LS139
- added U32, U33, U34, U35: SBC18-11EGWA, Display_7Segment:SBC18-11SURKCGKWA, symbol Display_Character:SBC18-11EGWA
Connections:
- net +5V: now also C10.1, C11.1, C12.1, C13.1, C14.1, C15.1, C16.1, C17.1, C18.1, C19.1, C20.1, C21.1, C22.1, C23.1, C24.1, C25.1, C26.1, C27.1, C28.1, C29.1, C30.1, C31.1, C32.1, C33.1, C34.1, C35.1, C36.1, C37.1, C8.1, C9.1, R19.1, U21.1 (MR), U21.20 (VCC), U28.21 (~{WE}), U28.24 (VCC), U29.4 (~{RST}), U29.8 (VCC), U30.12 (K2), U30.16 (K1), U30.2 (~{PRE}1), U30.3 (~{CLR}1), U30.4 (J1), U30.5 (VCC), U30.7 (~{PRE}2), U30.8 (~{CLR}2), U30.9 (J2), U31.16 (VCC)
- net BUS1: now also U21.3 (D0)
- net BUS2: now also U21.4 (D1)
- net BUS3: now also U21.7 (D2)
- net BUS4: now also U21.8 (D3)
- net BUS5: now also U21.13 (D4)
- net BUS6: now also U21.14 (D5)
- net BUS7: now also U21.17 (D6)
- net BUS8: now also U21.18 (D7)
- net GND: now also C10.2, C11.2, C12.2, C13.2, C14.2, C15.2, C16.2, C17.2, C18.2, C20.2, C21.2, C22.2, C23.2, C24.2, C25.2, C26.2, C27.2, C28.2, C29.2, C3.2, C30.2, C31.2, C32.2, C33.2, C34.2, C35.2, C36.2, C37.2, C7.1, C8.2, C9.2, U21.10 (GND), U28.12 (GND), U28.18 (~{CS}), U28.19 (A10), U28.20 (~{OE}), U29.1 (GND), U30.13 (GND), U31.1 (~{G}1), U31.8 (GND)
- new net: R19.2, R20.1, U29.7 (DISCH)
- new net: R17.1, U28.14 (D4)
- new net: C7.2, U29.5 (CONT)
- new net: R11.2, U28.9 (D0)
- new net: C3.1, R20.2, U29.2 (TRIG), U29.6 (THRES)
- new net: R14.1, U28.17 (D7)
- new net: R13.2, U28.11 (D2)
- new net: R12.2, U28.10 (D1)
- new net: R15.1, U28.16 (D6)
- new net: R18.1, U28.13 (D3)
- new net: R16.1, U28.15 (D5)
- new net CLK1: U29.3 (OUT), U30.1 (CLK1)
- new net CLK2: U28.23 (A8), U30.15 (Q1), U30.6 (CLK2), U31.2 (1A)
- new net CONQ_0: U21.2 (Q0), U28.8 (A0)
- new net CONQ_1: U21.5 (Q1), U28.7 (A1)
- new net CONQ_2: U21.6 (Q2), U28.6 (A2)
- new net CONQ_3: U21.9 (Q3), U28.5 (A3)
- new net CONQ_4: U21.12 (Q4), U28.4 (A4)
- new net CONQ_5: U21.15 (Q5), U28.3 (A5)
- new net CONQ_6: U21.16 (Q6), U28.2 (A6)
- new net CONQ_7: U21.19 (Q7), U28.1 (A7)
- new net JKQ2: U28.22 (A9), U30.11 (Q2), U31.3 (1B)
- new net OI: U21.11 (CP)
- new net SEG1: R11.1, U32.7 (A), U33.7 (A), U34.7 (A), U35.7 (A)
- new net SEG2: R12.1, U32.6 (B), U33.6 (B), U34.6 (B), U35.6 (B)
- new net SEG3: R13.1, U32.4 (C), U33.4 (C), U34.4 (C), U35.4 (C)
- new net SEG4: R18.2, U32.3 (D), U33.3 (D), U34.3 (D), U35.3 (D)
- new net SEG5: R17.2, U32.2 (E), U33.2 (E), U34.2 (E), U35.2 (E)
- new net SEG6: R16.2, U32.9 (F), U33.9 (F), U34.9 (F), U35.9 (F)
- new net SEG7: R15.2, U32.10 (G), U33.10 (G), U34.10 (G), U35.10 (G)
- new net SEG8: R14.2, U32.8 (DP), U33.8 (DP), U34.8 (DP), U35.8 (DP)
- new net SEGCC1: U31.4 (1Y0), U32.5 (CC)
- new net SEGCC2: U31.5 (1Y1), U33.5 (CC)
- new net SEGCC3: U31.6 (1Y2), U34.5 (CC)
- new net SEGCC4: U31.7 (1Y3), U35.5 (CC)
Other:
- moved on the sheet: D2, R7, U1, U2, U20, U24, U26, U7

Commit message: Add files via upload
Parts:
- added C38, C39, C40: 100nF, symbol Device:C_Small
- added U36: 74LS161, symbol 8-bit ICs:74LS161
- added U38: 28C16, symbol 8-bit ICs:28C16
- added U39: 74LS04, symbol 8-bit ICs:74LS04
- added U40: 74LS00, symbol 8-bit ICs:74LS00
- added U41: 74LS08, symbol 8-bit ICs:74LS08
- added U42: 74LS245, symbol 8-bit ICs:74LS245
- added U43, U44: 74LS173, symbol 8-bit ICs:74LS173
Connections:
- net +5V: now also C38.1, C39.1, C40.1, U36.10 (ENT), U36.16 (VCC), U36.7 (ENP), U36.9 (~{LOAD}), U38.21 (~{WE}), U38.24 (VCC), U39.14 (VCC), U40.14 (VCC), U41.14 (VCC), U42.1 (DIR), U42.20 (VCC), U43.16 (VCC), U44.16 (VCC)
- net A1: now also U42.2 (A1), U43.3 (1Q)
- net A2: now also U42.3 (A2), U43.4 (2Q)
- net A3: now also U42.4 (A3), U43.5 (3Q)
- net A4: now also U42.5 (A4), U43.6 (4Q)
- net A5: now also U38.5 (A3), U42.6 (A5), U44.3 (1Q)
- net A6: now also U38.4 (A4), U42.7 (A6), U44.4 (2Q)
- net A7: now also U38.3 (A5), U42.8 (A7), U44.5 (3Q)
- net A8: now also U38.2 (A6), U42.9 (A8), U44.6 (4Q)
- net BUS1: now also U42.18 (B1), U43.14 (1D)
- net BUS2: now also U42.17 (B2), U43.13 (2D)
- net BUS3: now also U42.16 (B3), U43.12 (3D)
- net BUS4: now also U42.15 (B4), U43.11 (4D)
- net BUS5: now also U42.14 (B5), U44.14 (1D)
- net BUS6: now also U42.13 (B6), U44.13 (2D)
- net BUS7: now also U42.12 (B7), U44.12 (3D)
- net BUS8: now also U42.11 (B8), U44.11 (4D)
- net CARRY: now also U38.1 (A7)
- net CLK: now also U36.2 (CLK), U43.7 (CLK), U44.7 (CLK)
- net GND: now also C19.2, C38.2, C39.2, C40.2, U36.3 (A), U36.4 (B), U36.5 (C), U36.6 (D), U36.8 (GND), U38.12 (GND), U38.18 (~{CS}), U38.19 (A10), U38.20 (~{OE}), U38.22 (A9), U39.7 (GND), U40.7 (GND), U41.7 (GND), U42.10 (GND), U43.1 (M), U43.15 (CLR), U43.2 (N), U43.8 (GND), U44.1 (M), U44.15 (CLR), U44.2 (N), U44.8 (GND)
- net HALT_IN: now also U38.9 (D0)
- new net CONQA: U36.14 (QA), U38.8 (A0)
- new net CONQB: U36.13 (QB), U38.7 (A1)
- new net CONQC: U36.12 (QC), U38.6 (A2)
- new net CONQD: U36.11 (QD)
- new net ~{II}: U43.10 (~{G2}), U43.9 (~{G1}), U44.10 (~{G2}), U44.9 (~{G1})
- new net ~{IO}: U42.19 (~{OE})
- no-connect marks 42 -> 43
Other:
- note added: "Instruction Register"
- moved on the sheet: C1, C2, C30, C31, C32, C33, C34, C35, C36, C37, C4, C5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

Commit message: Add files via upload
Parts:
- added C41, C42, C43, C44, C45, C46, C47, C48: 100nF, symbol Device:C_Small
- added U37: 28C16, symbol 8-bit ICs:28C16
- added U45: 74LS173, symbol 8-bit ICs:74LS173
Connections:
- net +5V: now also C41.1, C42.1, C43.1, C44.1, C45.1, C46.1, C47.1, C48.1, U37.21 (~{WE}), U37.24 (VCC), U45.16 (VCC)
- net A5: now also U37.5 (A3)
- net A6: now also U37.4 (A4)
- net A7: now also U37.3 (A5)
- net A8: now also U37.2 (A6)
- net CARRY: now also U45.14 (1D); no longer U38.1 (A7)
- net CE: now also U37.14 (D4)
- net CLK: now also U45.7 (CLK)
- net CONQA: now also U37.8 (A0)
- net CONQB: now also U40.1 (1A), U37.7 (A1)
- net CONQC: now also U40.2 (1B), U37.6 (A2)
- net GND: now also C41.2, C42.2, C43.2, C44.2, C45.2, C46.2, C47.2, C48.2, U37.12 (GND), U37.18 (~{CS}), U37.19 (A10), U37.20 (~{OE}), U37.22 (A9), U45.10 (~{G2}), U45.8 (GND), U45.9 (~{G1})
- net OI: now also U37.13 (D3)
- net RI: now also U38.11 (D2)
- net RO: now also U38.13 (D3)
- net MI: now reaches U38.10 (D1)
- net IO: now reaches U38.14 (D4)
- net II: now reaches U38.15 (D5)
- net AI: now reaches U38.16 (D6)
- net A0: now reaches U38.17 (D7)
- net ZF: now reaches U38.23 (A8)
- net ZF: now also U37.23 (A8), U45.13 (2D)
- net InCouRST: now reaches U40.3 (1Y)
- net InCouRST: now also U36.1 (~{CLR})
- net MAR_RST renamed RAM_RST
- new net BI: U37.11 (D2)
- new net CF: U37.1 (A7), U38.1 (A7)
- new net CO: U37.15 (D5)
- new net EO: U37.9 (D0)
- new net FI: U37.17 (D7), U45.1 (M), U45.2 (N)
- new net FR_RST: U45.15 (CLR)
- new net J: U37.16 (D6)
- new net SU: U37.10 (D1)
Other:
- moved on the sheet: C3, C7, C8, C9, R19, R20, U21, U29, U30, U36, U38, U39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
